File: ESP32-Liligo-Disp-Temp-Hat.kicad_pcb (KiCad board)
At the start: 4 copper layers, 48.3 x 99.7 mm, 45 parts, among them J1 Conn_02x11_Odd_Even, J10 Conn_01x09, J11 Conn_01x02, J2 Conn_01x02, J3 Conn_01x02, J4 Conn_01x02, J5 Conn_01x02, J6 Conn_01x02, J7 Conn_01x02, J8 Conn_01x02, J9 Conn_01x02, U1 TMUX1108PW, U2 MAX31856, U3 TMUX1108PW, U4 PCF8574ATS, U5 74LVC1G04, U6 INA215DCK

Commit message: Finish routing
Parts:
- moved J11 3.53 mm to (123.7, 141.6)
- moved R6 3.53 mm to (117.3, 144.5)
- moved C14 3.53 mm to (113.9, 146.1)
- moved U6 3.53 mm to (113.8, 142.4)
- moved JP3 0.26 mm to (119.1, 106.2)
Routing:
- net I2C_SCL: track 0.00 -> 94.6 mm
- net I2C_SDA: track 0.00 -> 77.5 mm, vias 0 -> 1
- net TC7+: track 0.00 -> 77.4 mm, vias 0 -> 1
- net EXPANDER_INT: track 0.00 -> 73.7 mm
- net JOYSTICK_CONFIRM: track 0.00 -> 72.0 mm, vias 0 -> 1
- net JOYSTICK_BACK: track 0.00 -> 65.2 mm, vias 0 -> 1
- net TC6+: track 0.00 -> 65.1 mm, vias 0 -> 1
- net TC7-: track 0.00 -> 58.0 mm
- net TC5+: track 0.00 -> 52.0 mm, vias 0 -> 1
- net TC_CS: track 0.00 -> 50.1 mm
- net TC_A0: track 0.00 -> 47.7 mm
- net TC_SCK: track 0.00 -> 47.7 mm
- net TC6-: track 0.00 -> 46.5 mm
- net TC_MISO: track 0.00 -> 45.7 mm, vias 0 -> 1
- net TC_MOSI: track 0.00 -> 43.6 mm, vias 0 -> 1
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
Commit message: Add onewire connector
Parts:
- added J12: Conn_01x03_MountingPin, Connector_JST:JST_PH_S3B-PH-SM4-TB_1x03-1MP_P2.00mm_Horizontal, F.Cu at (110.1, 87.7)
Connections:
- J1 pad 10: unconnected-(J1-Pin_10-Pad10) -> ONEWIRE
Routing:
- net ONEWIRE: track 0.00 -> 76.9 mm, vias 0 -> 1
- net GND: track 40.9 -> 48.7 mm, vias 26 -> 29
- net VCC: track 29.0 -> 32.4 mm, vias 12 -> 13
