File: ESP32-Liligo-Disp-Temp-Hat.kicad_sch (KiCad schematic)
At the start: 45 parts, among them J1 Conn_02x11_Odd_Even, J10 Conn_01x09, J11 Conn_01x02, J2 Conn_01x02, J3 Conn_01x02, J4 Conn_01x02, J5 Conn_01x02, J6 Conn_01x02, J7 Conn_01x02, J8 Conn_01x02, J9 Conn_01x02, U1 TMUX1108PW, U2 MAX31856, U3 TMUX1108PW, U4 PCF8574ATS, U5 74LVC1G04, U6 INA215DCK

Commit message: Add onewire connector
Parts:
- added J12: Conn_01x03_MountingPin, Connector_JST:JST_PH_S3B-PH-SM4-TB_1x03-1MP_P2.00mm_Horizontal, symbol Connector_Generic_MountingPin:Conn_01x03_MountingPin
Connections:
- net GND: now also J12.2 (Pin_2), J12.MP (MountPin)
- net VCC: now also J12.3 (Pin_3)
- net ONEWIRE: now reaches J1.10 (Pin_10)
- net ONEWIRE: now also J12.1 (Pin_1)
- no-connect marks 6 -> 5
